Commit message: remove chest joint to simplify

File: learning_urdf/urdf/NextageOpen_LeftArmOnly.urdf (robot description, URDF)
Before this commit: robot NextageOpen, 8 links, 7 joints
Links:
- removed link CHEST_JOINT0_Link
Joints:
- removed joint CHEST_JOINT0
- joint LARM_JOINT0: parent CHEST_JOINT0_Link -> WAIST

Commit message: add left arm link geometries in urdf

File: learning_urdf/urdf/NextageOpen_LeftArmOnly.urdf (robot description, URDF)
Before this commit: robot NextageOpen, 7 links, 6 joints
Links:
- link LARM_JOINT0_Link: mass None -> 1.32626; geometry collision mesh filename=package://nextage_description/urdf/meshes/LARM_JOINT0_Link_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 scale=1 1 1; visual mesh filename=package://nextage_description/urdf/meshes/LARM_JOINT0_Link_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 scale=1 1 1
- link LARM_JOINT1_Link: mass None -> 1.14898; geometry collision mesh filename=package://nextage_description/urdf/meshes/LARM_JOINT1_Link_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 scale=1 1 1; visual mesh filename=package://nextage_description/urdf/meshes/LARM_JOINT1_Link_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 scale=1 1 1
- link LARM_JOINT2_Link: mass None -> 0.577518; geometry collision mesh filename=package://nextage_description/urdf/meshes/LARM_JOINT2_Link_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 scale=1 1 1; visual mesh filename=package://nextage_description/urdf/meshes/LARM_JOINT2_Link_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 scale=1 1 1
- link LARM_JOINT3_Link: mass None -> 0.457418; geometry collision mesh filename=package://nextage_description/urdf/meshes/LARM_JOINT3_Link_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 scale=1 1 1; visual mesh filename=package://nextage_description/urdf/meshes/LARM_JOINT3_Link_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 scale=1 1 1
- link LARM_JOINT4_Link: mass None -> 0.418434; geometry collision mesh filename=package://nextage_description/urdf/meshes/LARM_JOINT4_Link_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 scale=1 1 1; visual mesh filename=package://nextage_description/urdf/meshes/LARM_JOINT4_Link_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 scale=1 1 1
- link LARM_JOINT5_Link: mass None -> 1.05156; geometry collision mesh filename=package://nextage_description/urdf/meshes/LARM_JOINT5_Link_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 scale=1 1 1; visual mesh filename=package://nextage_description/urdf/meshes/LARM_JOINT5_Link_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 scale=1 1 1
